File: PCB/MIDI-keypad.kicad_pcb (KiCad board)
At the start: 2 copper layers, 97 x 95 mm, 11 parts, among them J1 Capacitive Touch Buttons, SW1 SW_Push, SW2 SW_Push, SW3 SW_Push, SW4 RotaryEncoder_Switch_MP, U1 Waveshare ESP32-S3-ZERO

Commit message: finishing silkscreen art
Parts:
- added G***: LOGO, LOGO, F.Cu at (107.0, 63.2)
- added G***: LOGO, LOGO, F.Cu at (140.6, 62.3)
- added G***: LOGO, LOGO, B.Cu at (147.4, 139.5)
- added G***: LOGO, LOGO, B.Cu at (148.2, 104.7)
Other:
- board text added: "By: Kai Pereira"
- board text added: "kaipereira.com"
