File: PCB/MIDI-keypad.kicad_pcb (KiCad board)
At the start: 2 copper layers, 97 x 95 mm, 15 parts, among them J1 Capacitive Touch Buttons, SW1 SW_Push, SW2 SW_Push, SW3 SW_Push, SW4 RotaryEncoder_Switch_MP, U1 Waveshare ESP32-S3-ZERO

Commit message: fixing analog slider pins
Connections:
- U1 pad 1: /ENC1_A -> /SLIDE2
- U1 pad 2: /ENC1_B -> /SLIDE1
- U1 pad RX: /SLIDE2 -> /ENC1_B
- U1 pad TX: /SLIDE1 -> /ENC1_A
Routing:
- net GND: track 239.7 -> 220.5 mm
- net /ENC1_B: track 61.0 -> 79.3 mm
- net /ENC1_A: track 62.0 -> 76.7 mm
- net /SLIDE1: track 59.6 -> 50.0 mm
- net +3V3: track 183.4 -> 179.0 mm
- net /SLIDE2: track 45.3 -> 41.5 mm
